File: eagle/rapi-receiver/receiver.brd (EAGLE design)
At the start: 65 x 21 mm, 26 parts, among them IC100 CC110L_RTK_20, IC200 Value, IC300 CAT24C32WI-GT3, IC400 Value, X120 CRYSTAL.3.2X2.5MM

Commit message: CHG: updated lib, schematics and boards
Parts:
- U$1: value ANTENNA868W3013-INV -> (none)
