File: eagle/rapi-receiver/receiver.sch (EAGLE design)
At the start: 57 parts, among them IC100 LPS25H, IC200 Value, IC300 CC110L_RTK_20, IC400 Value, IC500 MSP430FR5720_RGE_24, IC600 Value, IC700 Value, X320 CRYSTAL.3.2X2.5MM

Commit message: CHG: updated lib, schematics and boards
Parts:
- removed !PROG, BAT: (no value), pinhead:PINHD-1X2
- removed ADRESS: SWS003, smd-special:SWS003
- removed C201, C241: 4u7, rcl:C-EUC0603
- removed C210: 22u, rcl:C-EUC0603
- removed C240: 10n, rcl:C-EUC0603
- removed C301, C302, C310, C500, C501, C600, C700: 100n, rcl:C-EUC0603
- removed C320, C321: 15p, rcl:C-EUC0603
- removed C350: 1p8, rcl:C-EUC0603K
- removed C351: 100p, rcl:C-EUC0603
- removed C352: 100p, rcl:C-EUC0603K
- removed C510: 470n, rcl:C-EUC0603
- removed F300: 2450BM15A0002, johanson-technology:2450BM15A0002
- removed IC500: MSP430FR5720_RGE_24, weather_station:MSP430FR5720_RGE_24
- removed IC600: Value, weather_station:TMP102AQDRLRQ1
- removed IC700: Value, weather_station:TPL5110DDCR
- removed L200: 22u, rcl:L-EUL3225P
- removed L210: 10u, rcl:L-EUL3225P
- removed L350: 5n6, rcl:L-EUL2012C
- removed LINK: (no value), pinhead:PINHD-1X6
- removed PROG: (no value), pinhead:PINHD-1X4
- removed R200, R510, R511, R711: DNB, rcl:R-EU_R0603
- removed R201, R710: 0, rcl:R-EU_R0603
- removed R210: 13M, rcl:R-EU_R0603
- removed R211: 5M62, rcl:R-EU_R0603
- removed R220: 100k, rcl:R-EU_R0603
- removed R221: 8M7, rcl:R-EU_R0603
- removed R222: 4M2, rcl:R-EU_R0603
- removed R230: 7M8, rcl:R-EU_R0603
- removed R231: 5M2, rcl:R-EU_R0603
- removed R500: 10k, rcl:R-EU_R0603
- removed R700: 18k75, rcl:R-EU_R0603
- removed S1: SKHMPSE010, switch:SKHMPSE010
- removed X320: CRYSTAL.3.2X2.5MM, abracon:CRYSTAL.3.2X2.5MM
- added !WP: (no value), pinhead:PINHD-1X2
- added C102, C110: 100n, rcl:C-EUC0603
- added C120, C121: 15p, rcl:C-EUC0603
- added C150: 1p8, rcl:C-EUC0603K
- added C151: 100p, rcl:C-EUC0603
- added C152: 100p, rcl:C-EUC0603K
- added F100: 2450BM15A0002, johanson-technology:2450BM15A0002
- added L150: 5n6, rcl:L-EUL2012C
- added PCB1: RPI2, weather_station:RPI2
- added R100: 56k, rcl:R-EU_R0603
- added R310, R311: 3k9, rcl:R-EU_R0603
- added X120: CRYSTAL.3.2X2.5MM, abracon:CRYSTAL.3.2X2.5MM
- C101: value 4u7 -> 100n
- C200: value 10n -> 100n
- IC100: value LPS25H -> CC110L_RTK_20; device weather_station:LPS25H -> weather_station:CC110L_RTK_20
- IC200: device weather_station:BQ25570RGRR -> weather_station:HDC1000YPAR
- IC300: value CC110L_RTK_20 -> CAT24C32WI-GT3; device weather_station:CC110L_RTK_20 -> weather_station:CAT24C32WI-GT3
- IC400: device weather_station:HDC1000YPAR -> weather_station:TMP102AQDRLRQ1
- R300: value 56k -> 1k
- U$1: value ANTENNA868W3013-INV -> (none)
Connections:
- removed net !CC110L_CS: IC300.CSN, IC500.PJ.0/TDO/TB0OUTH/SMCLK/CD6
- removed net !LINK_INT: IC500.P1.4/TB0.1/UCA0STE/A4*/CD4, LINK.6
- removed net !MSP430_RST: IC500.*RST/NMI/SBWTDIO, PROG.3, R500.1
- removed net ADRESS_0: ADRESS.6, IC500.PJ.1/TDI/TCLK/MCLK/CD7
- removed net ADRESS_1: ADRESS.5, IC500.PJ.2/TMS/ACLK/CD8
- removed net BQ25570_VBAT_OK: IC200.VBAT_OK, IC500.P1.3/TA1.2/UCB0STE/A3*/CD3
- removed net BQ25570_VOUT_EN: IC200.VOUT_EN, R200.2, R201.1
- removed net BQ25570_VSTOR: C240.2, C241.2, C700.1, IC200.VOC_SAMP, IC200.VSTOR, IC700.VDD, R200.1, R710.2, S1.2.1, S1.2.2
- removed net DEVICE: ADRESS.4, IC500.PJ.3/TCK/CD9
- removed net LPS25H_INT: IC100.INT, IC500.P1.1/TA0.2/TA1CLK/CDOUT/A1*/CD1/VEREF+*
- removed net MSP430_CLK: IC300.SCLK1, IC500.P1.5/TB0.2/UCA0CLK/A5*/CD5
- removed net MSP430_MISO: IC300.SO, IC500.P2.1/UCA0RXD/UCA0SOMI/TB0.0
- removed net MSP430_MOSI: IC300.SI, IC500.P2.0/UCA0TXD/UCA0SIMO/TB0CLK/ACLK
- removed net MSP430_P2.2: IC500.P2.2/UCB0CLK, R510.1, R511.1
- removed net MSP430_SCL: IC100.SCL, IC400.SCL, IC500.P1.7/UCB0SOMI/UCB0SCL/TA1.0, IC600.SCL, LINK.5
- removed net MSP430_SDA: IC100.SDA, IC400.SDA, IC500.P1.6/UCB0SIMO/UCB0SDA/TA0.0, IC600.SDA, LINK.4
- removed net MSP430_TEST: IC500.TEST/SBWTCK, PROG.2
- removed net MSP430_VCORE: C510.1, IC500.VCORE
- removed net N$14: IC200.OK_HYST, R220.1, R221.2
- removed net N$15: IC200.VRDIV, R210.1, R220.2, R230.2
- removed net N$16: IC200.VBAT_OV, R210.2, R211.2
- removed net N$17: IC200.OK_PROG, R221.1, R222.2
- removed net N$18: IC200.LBOOST, L200.2
- removed net N$19: C200.1, IC200.VREF_SAMP
- removed net N$21: IC200.VOUT_SET, R230.1, R231.2
- removed net N$22: !PROG.2, C210.1, IC200.VOUT, L210.2
- removed net N$25: IC200.LBUCK, L210.1
- removed net N$26: BAT.1, IC200.VBAT
- removed net N$7: IC700.DELAY_M_DRV, R700.1, S1.1.1, S1.1.2
- removed net SOLAR_P: C201.1, IC200.VIN_DC, L200.1, LINK.1
- removed net TPL5010_RST_N: IC700.EN_ONE_SHOT, R710.1, R711.2
- removed net TPL5111_DONE: IC500.PJ.5/XOUT, IC700.DONE
- removed net TPL5111_DRV: IC700.DRV, R201.2, R510.2
- new net +5V: PCB1.5V@2, PCB1.5V@4
- new net CC110L_CS: IC100.CSN, PCB1.GPIO15
- new net N$33: F100.UNBAL, L150.1
- new net RB2_ID_SC: IC300.SCL, PCB1.ID_SC*, R310.1
- new net RB2_ID_SD: IC300.SDA, PCB1.ID_SD*, R311.1
- new net RB2_MISO: IC100.SO, PCB1.GPIO9
- new net RB2_MOSI: IC100.SI, PCB1.GPIO10
- new net RB2_SCL: IC200.SCL, IC400.SCL, PCB1.GPIO3
- new net RB2_SCLK: IC100.SCLK1, PCB1.GPIO11
- new net RB2_SDA: IC200.SDA, IC400.SDA, PCB1.GPIO2
- net !HDC1000_INT: now also IC200.DRDY_N, PCB1.GPIO4; no longer IC400.DRDY_N, IC500.P1.2/TA1.1/TA0CLK/CDOUT/A2*/CD2
- net !TMP102_ALERT: now also IC400.ALERT, PCB1.GPIO14; no longer IC500.P1.0/TA0.1/DMAE0/RTCCLK/A0*/CD0/VEREF-*, IC600.ALERT
- net CC110L_GDO0: now also IC100.GDO0, PCB1.GPIO18; no longer IC300.GDO0, IC500.PJ.4/XIN
- net CC110L_GDO2: now also IC100.GDO2, PCB1.GPIO23; no longer IC300.GDO2, R511.2
- net GND: now also !WP.1, C102.2, C110.2, C120.2, C121.2, C150.1, C152.2, C300.1, F100.GND@1, F100.GND@2, F100.GND@3, IC100.EPAD, IC100.GND, IC100.GND_2, IC200.ADR0, IC200.ADR1, IC200.GND, IC300.A0, IC300.A1, IC300.A2, IC300.VSS, IC400.ADD0, PCB1.GND@14, PCB1.GND@20, PCB1.GND@25, PCB1.GND@30, PCB1.GND@34, PCB1.GND@39, PCB1.GND@6, PCB1.GND@9, R100.1, X120G$2.P$1; no longer ADRESS.1, ADRESS.2, BAT.2, C201.2, C210.2, C240.1, C241.1, C300.2, C301.2, C302.2, C310.2, C320.2, C321.2, C350.1, C352.2, C500.2, C501.2, C510.2, C600.2, C700.2, F300.GND@1, F300.GND@2, F300.GND@3, IC100.GND@1, IC100.GND@2, IC100.RGND, IC100.SA0, IC200.EN_N, IC200.NC, IC200.NC_2, IC200.PAD, IC200.VSS, IC200.VSS_2, IC300.EPAD, IC300.GND, IC300.GND_2, IC400.ADR0, IC400.ADR1, IC500.AVSS, IC500.DVSS, IC500.EPAD, IC600.ADD0, IC600.GND, IC700.GND, LINK.2, PROG.4, R211.1, R222.1, R231.1, R300.1, R700.2, R711.1, S1.SH, X320G$2.P$1
- net N$1: now also !WP.2, IC300.WP, R300.1; no longer C351.1, C352.1, U$1.P$1
- net N$2: now also C151.1, C152.1, U$1.P$1; no longer F300.UNBAL, L350.1
- net N$29: now also C120.1, IC100.XOSC_Q1, X120G$1.2; no longer C320.1, IC300.XOSC_Q1, X320G$1.2
- net N$34: now also F100.BAL@1, IC100.RF_N; no longer F300.BAL@1, IC300.RF_N
- net N$35: now also F100.BAL@2, IC100.RF_P; no longer F300.BAL@2, IC300.RF_P
- net N$36: now also C150.2, C151.2, L150.2; no longer C350.2, C351.2, L350.2
- net N$40: now also C110.1, IC100.DCOUPL; no longer C310.1, IC300.DCOUPL
- net N$41: now also IC100.RBIAS, R100.2; no longer IC300.RBIAS, R300.2
- net N$49: now also C121.1, IC100.XOSC_Q2, X120G$1.1; no longer C321.1, IC300.XOSC_Q2, X320G$1.1
- net VCC: now also C102.1, C200.1, C300.2, IC100.AVDD, IC100.AVDD_2, IC100.AVDD_3, IC100.AVDD_4, IC100.DGUARD, IC100.DVDD, IC200.VDD, IC300.VCC, IC400.V+, PCB1.3V3@1, PCB1.3V3@17, R300.2, R310.2, R311.2; no longer !PROG.1, C300.1, C301.1, C302.1, C500.1, C501.1, C600.1, IC100.CS, IC100.VDD, IC100.VDD_IO, IC300.AVDD, IC300.AVDD_2, IC300.AVDD_3, IC300.AVDD_4, IC300.DGUARD, IC300.DVDD, IC400.VDD, IC500.AVCC, IC500.DVCC, IC600.V+, LINK.3, PROG.1, R500.2
