File: eagle/outdoorsensor/outdoor-sensor.brd (EAGLE design)
At the start: 40.5 x 60.2 mm, 61 parts, among them IC100 LPS25H, IC200 Value, IC300 CC110L_RTK_20, IC400 Value, IC500 MSP430FR5739_RHA_40, IC600 Value, IC700 Value, IC800 MAX17048X+, X320 CRYSTAL.3.2X2.5MM

Commit message: CHG: Updated schematics and layout
Parts:
- R210: value 13M -> 7M32
- R230: value 7M8 -> 8M3
- R231: value 5M2 -> 4M7
Routing:
- net GND: vias 589 -> 588
Changed lines of the file:
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@@
 <?xml version="1.0" encoding="utf-8"?>
 <!DOCTYPE eagle SYSTEM "eagle.dtd">
-<eagle version="6.5.0">
+<eagle version="7.4.0">
 <drawing>
 <settings>
@@
 <layer number="54" name="bGND_GNDA" color="1" fill="9" visible="no" active="no"/>
 <layer number="56" name="wert" color="7" fill="1" visible="no" active="no"/>
-<layer number="90" name="Modules" color="5" fill="1" visible="no" active="yes"/>
+<layer number="90" name="Modules" color="5" fill="1" visible="no" active="no"/>
 <layer number="91" name="Nets" color="2" fill="1" visible="no" active="no"/>
 <layer number="92" name="Busses" color="1" fill="1" visible="no" active="no"/>
@@
 <pass name="Default">
 <param name="RoutingGrid" value="50mil"/>
+<param name="AutoGrid" value="1"/>
+<param name="Efforts" value="0"/>
+<param name="TopRouterVariant" value="1"/>
 <param name="tpViaShape" value="round"/>
 <param name="PrefDir.1" value="|"/>
@@
 <attribute name="MPN" value="" x="37.1475" y="10.16" size="1.778" layer="27" rot="R180" display="off"/>
 </element>
-<element name="R210" library="rcl" package="R0603" value="13M" x="36.5125" y="21.9075" smashed="yes">
+<element name="R210" library="rcl" package="R0603" value="7M32" x="36.5125" y="21.9075" smashed="yes">
 <attribute name="NAME" x="36.5125" y="20.32" size="1.016" layer="25" align="center"/>
 <attribute name="VALUE" x="35.8775" y="20.0025" size="1.27" layer="27"/>
@@
 <attribute name="MPN" value="" x="33.02" y="24.4475" size="1.778" layer="27" display="off"/>
 </element>
-<element name="R230" library="rcl" package="R0603" value="7M8" x="29.5275" y="21.9075" smashed="yes">
+<element name="R230" library="rcl" package="R0603" value="8M3" x="29.5275" y="21.9075" smashed="yes">
 <attribute name="NAME" x="29.5275" y="23.1775" size="1.016" layer="25" align="center"/>
 <attribute name="VALUE" x="28.8925" y="20.0025" size="1.27" layer="27"/>
@@
 <attribute name="MPN" value="" x="33.02" y="19.3675" size="1.778" layer="27" display="off"/>
 </element>
-<element name="R231" library="rcl" package="R0603" value="5M2" x="29.5275" y="19.3675" smashed="yes" rot="R180">
+<element name="R231" library="rcl" package="R0603" value="4M7" x="29.5275" y="19.3675" smashed="yes" rot="R180">
 <attribute name="NAME" x="29.5275" y="18.25625" size="1.016" layer="25" rot="R180" align="center"/>
 <attribute name="VALUE" x="30.1625" y="21.2725" size="1.27" layer="27" rot="R180"/>
@@
 <via x="5.3975" y="31.4325" extent="1-16" drill="0.3"/>
 <via x="4.1275" y="33.3375" extent="1-16" drill="0.3"/>
-<via x="6.19125" y="33.81375" extent="1-16" drill="0.3"/>
+<wire x1="6.19125" y1="33.81375" x2="6.19125" y2="33.81375" width="0" layer="19" extent="1-16"/>
 <via x="6.19125" y="34.76625" extent="1-16" drill="0.3"/>
 <via x="3.96875" y="37.1475" extent="1-16" drill="0.3"/>

Commit message: CHG: fixed some issuses on pcb
Parts:
- added R712: 100k, rcl:R0603
- moved R700 3.63 mm to (10.0, 50.2), turned to 0 degrees
Connections:
- net GND: now also R712.1
- net TPL5111_DONE: now also R712.2
- net TPL5111_DRV: no longer IC500.26
Routing:
- net TPL5111_DRV: track 40.6 -> 35.7 mm
- net N$7: track 22.9 -> 19.6 mm
Changed lines of the file:
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@@
 <attribute name="MPN" value="" x="31.59125" y="7.77875" size="1.778" layer="27" rot="R90" display="off"/>
 </element>
-<element name="R700" library="rcl" package="R0603" value="18k75" x="6.6675" y="51.59375" smashed="yes" rot="R90">
-<attribute name="NAME" x="4.92125" y="51.59375" size="1.016" layer="25" rot="R270" align="center"/>
-<attribute name="VALUE" x="8.5725" y="50.95875" size="1.27" layer="27" rot="R90"/>
-<attribute name="OC_FARNELL" value="unknown" x="6.6675" y="51.59375" size="1.778" layer="27" rot="R90" display="off"/>
-<attribute name="MF" value="" x="6.6675" y="51.59375" size="1.778" layer="27" rot="R90" display="off"/>
-<attribute name="MPN" value="" x="6.6675" y="51.59375" size="1.778" layer="27" rot="R90" display="off"/>
+<element name="R700" library="rcl" package="R0603" value="18k75" x="10.00125" y="50.165" smashed="yes">
+<attribute name="NAME" x="10.00125" y="51.91125" size="1.016" layer="25" rot="R180" align="center"/>
+<attribute name="VALUE" x="9.36625" y="48.26" size="1.27" layer="27"/>
+<attribute name="OC_FARNELL" value="unknown" x="10.00125" y="50.165" size="1.778" layer="27" display="off"/>
+<attribute name="MF" value="" x="10.00125" y="50.165" size="1.778" layer="27" display="off"/>
+<attribute name="MPN" value="" x="10.00125" y="50.165" size="1.778" layer="27" display="off"/>
 </element>
 <element name="R710" library="rcl" package="R0603" value="0" x="13.49375" y="46.99" smashed="yes" rot="R90">
@@
 <attribute name="NAME" x="16.51" y="9.525" size="1.016" layer="25" rot="R180" align="center"/>
 <attribute name="VALUE" x="20.32" y="11.43" size="1.27" layer="27" rot="R180"/>
+</element>
+<element name="R712" library="rcl" package="R0603" value="100k" x="8.89" y="43.97375">
+<attribute name="MPN" value="" x="8.89" y="43.97375" size="1.778" layer="27" display="off"/>
+<attribute name="OC_FARNELL" value="unknown" x="8.89" y="43.97375" size="1.778" layer="27" display="off"/>
+<attribute name="MF" value="" x="8.89" y="43.97375" size="1.778" layer="27" display="off"/>
 </element>
 </elements>
@@
 <contactref element="R700" pad="2"/>
 <contactref element="IC700" pad="2"/>
-<contactref element="S1" pad="5"/>
 <contactref element="R711" pad="1"/>
 <contactref element="C700" pad="2"/>
@@
 <via x="31.27375" y="59.53125" extent="1-16" drill="0.3"/>
 <via x="13.81125" y="45.085" extent="1-16" drill="0.3"/>
-<via x="5.55625" y="51.59375" extent="1-16" drill="0.3"/>
-<via x="11.1125" y="50.00625" extent="1-16" drill="0.3"/>
+<via x="5.55625" y="50.8" extent="1-16" drill="0.3"/>
+<via x="8.255" y="48.41875" extent="1-16" drill="0.3"/>
 <via x="12.85875" y="45.085" extent="1-16" drill="0.3"/>
 <wire x1="12.1800125" y1="14.105" x2="11.6799875" y2="14.105" width="0.254" layer="1"/>
@@
 <via x="28.575" y="37.62375" extent="1-16" drill="0.3"/>
 <via x="15.24" y="51.27625" extent="1-16" drill="0.3"/>
-<via x="8.09625" y="51.27625" extent="1-16" drill="0.3"/>
 <via x="25.24125" y="30.63875" extent="1-16" drill="0.3"/>
 <via x="24.60625" y="37.62375" extent="1-16" drill="0.3"/>
@@
 <via x="5.3975" y="31.4325" extent="1-16" drill="0.3"/>
 <via x="4.1275" y="33.3375" extent="1-16" drill="0.3"/>
-<wire x1="6.19125" y1="33.81375" x2="6.19125" y2="33.81375" width="0" layer="19" extent="1-16"/>
 <via x="6.19125" y="34.76625" extent="1-16" drill="0.3"/>
 <via x="3.96875" y="37.1475" extent="1-16" drill="0.3"/>
@@
 <via x="6.19125" y="29.68625" extent="1-16" drill="0.3"/>
 <via x="4.60375" y="32.22625" extent="1-16" drill="0.3"/>
-<via x="7.77875" y="43.18" extent="1-16" drill="0.3"/>
-<via x="8.41375" y="43.97375" extent="1-16" drill="0.3"/>
-<via x="9.2075" y="44.7675" extent="1-16" drill="0.3"/>
+<via x="8.09625" y="42.8625" extent="1-16" drill="0.3"/>
+<via x="4.60375" y="45.24375" extent="1-16" drill="0.3"/>
+<via x="6.985" y="44.7675" extent="1-16" drill="0.3"/>
 <via x="8.41375" y="45.56125" extent="1-16" drill="0.3"/>
 <via x="7.46125" y="45.72" extent="1-16" drill="0.3"/>
@@
 <via x="4.28625" y="48.41875" extent="1-16" drill="0.3"/>
 <via x="5.08" y="47.625" extent="1-16" drill="0.3"/>
-<via x="5.55625" y="50.8" extent="1-16" drill="0.3"/>
+<via x="6.50875" y="49.8475" extent="1-16" drill="0.3"/>
 <via x="4.7625" y="51.59375" extent="1-16" drill="0.3"/>
 <via x="0.635" y="52.86375" extent="1-16" drill="0.3"/>
@@
 <via x="4.92125" y="57.62625" extent="1-16" drill="0.3"/>
 <via x="6.6675" y="56.8325" extent="1-16" drill="0.3"/>
-<via x="10.795" y="49.37125" extent="1-16" drill="0.3"/>
-<via x="10.795" y="50.64125" extent="1-16" drill="0.3"/>
+<via x="7.77875" y="49.37125" extent="1-16" drill="0.3"/>
+<via x="9.2075" y="47.78375" extent="1-16" drill="0.3"/>
 <via x="11.7475" y="51.435" extent="1-16" drill="0.3"/>
-<via x="9.8425" y="51.435" extent="1-16" drill="0.3"/>
-<via x="9.2075" y="52.22875" extent="1-16" drill="0.3"/>
 <via x="12.7" y="52.3875" extent="1-16" drill="0.3"/>
 <via x="9.2075" y="53.18125" extent="1-16" drill="0.3"/>
@@
 <via x="10.95375" y="57.785" extent="1-16" drill="0.3"/>
 <via x="10.16" y="57.785" extent="1-16" drill="0.3"/>
+<via x="7.46125" y="52.705" extent="1-16" drill="0.3"/>
+<via x="7.46125" y="51.1175" extent="1-16" drill="0.3"/>
+<via x="8.09625" y="50.165" extent="1-16" drill="0.3"/>
+<contactref element="S1" pad="5"/>
+<contactref element="R712" pad="1"/>
 </signal>
 <signal name="LPS25H_INT">
@@
 <contactref element="R201" pad="2"/>
 <contactref element="IC700" pad="5"/>
-<contactref element="IC500" pad="26"/>
-<wire x1="8.9575125" y1="40.7575" x2="8.9575125" y2="42.7712625" width="0.3" layer="1"/>
-<wire x1="8.9575125" y1="42.7712625" x2="9.8425" y2="43.65625" width="0.3" layer="1"/>
-<wire x1="9.8425" y1="43.65625" x2="10.95375" y2="44.7675" width="0.3" layer="1"/>
 <wire x1="10.95375" y1="44.7675" x2="10.95375" y2="45.8216" width="0.3" layer="1"/>
 <wire x1="33.59875" y1="26.82875" x2="32.7025" y2="26.82875" width="0.3" layer="1"/>
@@
 <wire x1="15.71625" y1="41.43375" x2="14.2875" y2="42.8625" width="0.3" layer="1"/>
 <wire x1="14.2875" y1="42.8625" x2="11.43" y2="42.8625" width="0.3" layer="1"/>
-<wire x1="11.43" y1="42.8625" x2="11.1125" y2="43.18" width="0.3" layer="1"/>
-<wire x1="11.1125" y1="43.18" x2="10.95375" y2="43.33875" width="0.3" layer="1"/>
+<wire x1="11.43" y1="42.8625" x2="10.95375" y2="43.33875" width="0.3" layer="1"/>
 <wire x1="10.95375" y1="43.33875" x2="10.95375" y2="45.8216" width="0.3" layer="1"/>
 </signal>
@@
 <contactref element="IC700" pad="4"/>
 <contactref element="IC500" pad="27"/>
-<wire x1="8.4574875" y1="40.7575" x2="8.4574875" y2="43.0649875" width="0.3" layer="1"/>
-<wire x1="8.4574875" y1="43.0649875" x2="9.2075" y2="43.815" width="0.3" layer="1"/>
-<wire x1="9.2075" y1="43.815" x2="10.003740625" y2="44.611240625" width="0.3" layer="1"/>
-<wire x1="10.003740625" y1="44.611240625" x2="10.003740625" y2="45.8216" width="0.3" layer="1"/>
+<wire x1="8.4574875" y1="40.7575" x2="8.4574875" y2="41.7949875" width="0.3" layer="1"/>
+<wire x1="8.4574875" y1="41.7949875" x2="10.003740625" y2="43.341240625" width="0.3" layer="1"/>
+<wire x1="10.003740625" y1="43.341240625" x2="10.003740625" y2="44.1325" width="0.3" layer="1"/>
+<contactref element="R712" pad="2"/>
+<wire x1="10.003740625" y1="44.1325" x2="10.003740625" y2="45.8216" width="0.3" layer="1"/>
+<wire x1="9.74" y1="43.97375" x2="10.003740625" y2="44.1325" width="0.4064" layer="1"/>
 </signal>
 <signal name="!LINK_INT">
@@
 <contactref element="S1" pad="1"/>
 <contactref element="IC700" pad="3"/>
-<wire x1="10.003740625" y1="48.1584" x2="10.003740625" y2="50.321259375" width="0.4064" layer="1"/>
+<wire x1="10.003740625" y1="48.1584" x2="10.003740625" y2="49.312509375" width="0.4064" layer="1"/>
 <wire x1="7.865" y1="58.4475" x2="16.265" y2="58.4475" width="0.3" layer="1"/>
-<wire x1="10.003740625" y1="50.321259375" x2="9.8425" y2="50.4825" width="0.4064" layer="1"/>
-<wire x1="9.8425" y1="50.4825" x2="8.255" y2="52.07" width="0.4064" layer="1"/>
-<wire x1="8.255" y1="52.07" x2="8.255" y2="52.705" width="0.4064" layer="1"/>
-<via x="8.255" y="52.705" extent="1-16" drill="0.3"/>
-<wire x1="8.255" y1="52.705" x2="8.255" y2="55.245" width="0.4064" layer="16"/>
+<via x="8.255" y="51.1175" extent="1-16" drill="0.3"/>
+<wire x1="8.255" y1="51.1175" x2="8.255" y2="55.245" width="0.4064" layer="16"/>
 <via x="8.255" y="55.245" extent="1-16" drill="0.3"/>
 <wire x1="8.255" y1="55.245" x2="7.865" y2="55.635" width="0.4064" layer="1"/>
 <wire x1="7.865" y1="55.635" x2="7.865" y2="58.4475" width="0.4064" layer="1"/>
-<wire x1="6.6675" y1="50.74375" x2="6.92875" y2="50.4825" width="0.4064" layer="1"/>
-<wire x1="6.92875" y1="50.4825" x2="9.8425" y2="50.4825" width="0.4064" layer="1"/>
+<wire x1="10.003740625" y1="49.312509375" x2="9.15125" y2="50.165" width="0.4064" layer="1"/>
+<wire x1="8.255" y1="51.1175" x2="8.255" y2="51.06125" width="0.4064" layer="1"/>
+<wire x1="8.255" y1="51.06125" x2="9.15125" y2="50.165" width="0.4064" layer="1"/>
 </signal>
 <signal name="TPL5010_RST_N">
