File: eagle/outdoorsensor/outdoor-sensor.sch (EAGLE design)
At the start: 26 parts, among them IC100 CC110L_RTK_20, IC200 Value, IC300 CAT24C32WI-GT3, IC400 Value, X120 CRYSTAL.3.2X2.5MM

Commit message: CHG: updated lib, schematics and boards
Parts:
- removed !WP: (no value), pinhead:PINHD-1X2
- removed C102, C110: 100n, rcl:C-EUC0603
- removed C120, C121: 15p, rcl:C-EUC0603
- removed C150: 1p8, rcl:C-EUC0603K
- removed C151: 100p, rcl:C-EUC0603
- removed C152: 100p, rcl:C-EUC0603K
- removed F100: 2450BM15A0002, johanson-technology:2450BM15A0002
- removed L150: 5n6, rcl:L-EUL2012C
- removed PCB1: RPI2, weather_station:RPI2
- removed R100: 56k, rcl:R-EU_R0603
- removed R310, R311: 3k9, rcl:R-EU_R0603
- removed X120: CRYSTAL.3.2X2.5MM, abracon:CRYSTAL.3.2X2.5MM
- added !PROG: (no value), pinhead:PINHD-1X2
- added ADR0, ADR1, ADR2, DEV0, DEV1: (no value), jumper:SJW
- added BAT: (no value), pinhead:PINHD-1X2IPBS-102-01-T-S-GP
- added C201, C241: 4u7, rcl:C-EUC0603
- added C210: 22u, rcl:C-EUC0603
- added C240: 10n, rcl:C-EUC0603
- added C301, C302, C310, C500, C501, C600, C700, C800: 100n, rcl:C-EUC0603
- added C320, C321: 15p, rcl:C-EUC0603
- added C350: 1p8, rcl:C-EUC0603K
- added C351: 100p, rcl:C-EUC0603
- added C352: 100p, rcl:C-EUC0603K
- added C510: 470n, rcl:C-EUC0603
- added F300: 2450BM15A0002, johanson-technology:2450BM15A0002
- added IC500: MSP430FR5739_RHA_40, weather_station:MSP430FR5739_RHA_40
- added IC600: Value, weather_station:TMP102AQDRLRQ1
- added IC700: Value, weather_station:TPL5110DDCR
- added IC800: MAX17048X+, weather_station:MAX17048X+
- added L200: 22u, rcl:L-EUL3944
- added L210: 10u, rcl:L-EUM
- added L350: 5n6, rcl:L-EUL2012C
- added LINK: (no value), pinhead:PINHD-1X6
- added PROG: (no value), pinhead:PINHD-1X4
- added R200, R711: DNB, rcl:R-EU_R0603
- added R201, R710: 0, rcl:R-EU_R0603
- added R210: 13M, rcl:R-EU_R0603
- added R211: 5M62, rcl:R-EU_R0603
- added R220: 100k, rcl:R-EU_R0603
- added R221: 8M7, rcl:R-EU_R0603
- added R222: 4M2, rcl:R-EU_R0603
- added R230: 7M8, rcl:R-EU_R0603
- added R231: 5M2, rcl:R-EU_R0603
- added R500: 10k, rcl:R-EU_R0603
- added R700: 18k75, rcl:R-EU_R0603
- added S1: SKHMPSE010, switch:SKHMPSE010
- added X320: CRYSTAL.3.2X2.5MM, abracon:CRYSTAL.3.2X2.5MM
- C100, C300, C400: MF (none) -> STMICROELECTRONICS; MPN (none) -> STP100NF04; OC_FARNELL (none) -> 9935509
- C101: value 100n -> 4u7; OC_FARNELL (none) -> unknown
- C200: value 100n -> 10n; OC_FARNELL (none) -> unknown
- IC100: value CC110L_RTK_20 -> LPS25H; device weather_station:CC110L_RTK_20 -> weather_station:LPS25H; MF (none) -> STMICROELECTRONICS; MPN (none) -> LPS25HBTR; OC_FARNELL (none) -> 2474251
- IC200: device weather_station:HDC1000YPAR -> weather_station:BQ25570RGRR; OC_FARNELL (none) -> unknown
- IC300: value CAT24C32WI-GT3 -> CC110L_RTK_20; device weather_station:CAT24C32WI-GT3 -> weather_station:CC110L_RTK_20; OC_FARNELL (none) -> unknown
- IC400: device weather_station:TMP102AQDRLRQ1 -> weather_station:HDC1000YPAR; OC_FARNELL (none) -> unknown
- R300: value 1k -> 56k; OC_FARNELL (none) -> unknown
- U$1: OC_FARNELL (none) -> unknown
Connections:
- removed net +5V: PCB1.5V@2, PCB1.5V@4
- removed net CC110L_CS: IC100.CSN, PCB1.GPIO15
- removed net N$33: F100.UNBAL, L150.1
- removed net RB2_ID_SC: IC300.SCL, PCB1.ID_SC*, R310.1
- removed net RB2_ID_SD: IC300.SDA, PCB1.ID_SD*, R311.1
- removed net RB2_MISO: IC100.SO, PCB1.GPIO9
- removed net RB2_MOSI: IC100.SI, PCB1.GPIO10
- removed net RB2_SCL: IC200.SCL, IC400.SCL, PCB1.GPIO3
- removed net RB2_SCLK: IC100.SCLK1, PCB1.GPIO11
- removed net RB2_SDA: IC200.SDA, IC400.SDA, PCB1.GPIO2
- new net !CC110L_CS: IC300.CSN, IC500.P1.4/TB0.1/UCA0STE/A4*/CD4
- new net !LINK_INT: IC500.P1.0/TA0.1/DMAE0/RTCCLK/A0*/CD0/VEREF-*, LINK.6
- new net !MAX17048_ALERT: IC500.P4.1, IC800.*ALRT
- new net !MSP430_RST: IC500.*RST/NMI/SBWTDIO, PROG.3, R500.1
- new net ADRESS_0: ADR0.2, IC500.P1.3/TA1.2/UCB0STE/A3*/CD3
- new net ADRESS_1: ADR1.2, IC500.P3.3/A15*/CD15
- new net ADRESS_2: ADR2.2, IC500.P3.2/A14*/CD14
- new net BQ25570_VBAT_OK: IC200.VBAT_OK, IC500.P3.1/A13*/CD13
- new net BQ25570_VOUT_EN: IC200.VOUT_EN, R200.2, R201.1
- new net BQ25570_VSTOR: C240.2, C241.2, C700.1, IC200.VOC_SAMP, IC200.VSTOR, IC700.VDD, R200.1, R710.2, S1.2.1, S1.2.2
- new net DEVICE_0: DEV0.2, IC500.PJ.0/TDO/TB0OUTH/SMCLK/CD6
- new net DEVICE_1: DEV1.2, IC500.PJ.1/TDI/TCLK/TB1OUTH/MCLK/CD7
- new net LPS25H_INT: IC100.INT, IC500.P3.0/A12*/CD12
- new net MSP430_CLK: IC300.SCLK1, IC500.P1.5/TB0.2/UCA0CLK/A5*/CD5
- new net MSP430_MISO: IC300.SO, IC500.P2.1/TB2.1/UCA0RXD/UCA0SOMI/TB0.0
- new net MSP430_MOSI: IC300.SI, IC500.P2.0/TB2.0/UCA0TXD/UCA0SIMO/TB0CLK/ACLK
- new net MSP430_SCL: IC100.SCL, IC400.SCL, IC500.P1.7/TB1.2/UCB0SOMI/UCB0SCL/TA1.0, IC600.SCL, IC800.SCL, LINK.5
- new net MSP430_SDA: IC100.SDA, IC400.SDA, IC500.P1.6/TB1.1/UCB0SIMO/UCB0SDA/TA0.0, IC600.SDA, IC800.SDA, LINK.4
- new net MSP430_TEST: IC500.TEST/SBWTCK, PROG.2
- new net MSP430_VCORE: C510.1, IC500.VCORE
- new net N$14: IC200.OK_HYST, R220.1, R221.2
- new net N$15: IC200.VRDIV, R210.1, R220.2, R230.2
- new net N$16: IC200.VBAT_OV, R210.2, R211.2
- new net N$17: IC200.OK_PROG, R221.1, R222.2
- new net N$18: IC200.LBOOST, L200.2
- new net N$19: C200.1, IC200.VREF_SAMP
- new net N$21: IC200.VOUT_SET, R230.1, R231.2
- new net N$22: !PROG.2, C210.1, IC200.VOUT, L210.2
- new net N$25: IC200.LBUCK, L210.1
- new net N$7: IC700.DELAY_M_DRV, R700.1, S1.1.1, S1.1.2
- new net SOLAR_P: C201.1, IC200.VIN_DC, IC500.P2.3/TA0.0/UCA1STE/A6*/CD10, L200.1, LINK.1
- new net TPL5010_RST_N: IC700.EN_ONE_SHOT, R710.1, R711.2
- new net TPL5111_DONE: IC500.P3.7/TB2.2, IC700.DONE
- new net TPL5111_DRV: IC500.P3.6/TB2.1/TB1CLK, IC700.DRV, R201.2
- new net VBAT: BAT.1, C800.1, IC200.VBAT, IC500.P2.4/TA1.0/UCA1CLK/A7*/CD11, IC800.CELL, IC800.VDD
- net !HDC1000_INT: now also IC400.DRDY_N, IC500.P1.2/TA1.1/TA0CLK/CDOUT/A2*/CD2; no longer IC200.DRDY_N, PCB1.GPIO4
- net !TMP102_ALERT: now also IC500.P1.1/TA0.2/TA1CLK/CDOUT/A1*/CD1/VEREF+*, IC600.ALERT; no longer IC400.ALERT, PCB1.GPIO14
- net CC110L_GDO0: now also IC300.GDO0, IC500.P2.5/TB0.0/UCA1TXD/UCA1SIMO; no longer IC100.GDO0, PCB1.GPIO18
- net CC110L_GDO2: now also IC300.GDO2, IC500.P2.6/TB1.0/UCA1RXD/UCA1SOMI; no longer IC100.GDO2, PCB1.GPIO23
- net GND: now also ADR0.1, ADR1.1, ADR2.1, BAT.2, C201.2, C210.2, C240.1, C241.1, C300.2, C301.2, C302.2, C310.2, C320.2, C321.2, C350.1, C352.2, C500.2, C501.2, C510.2, C600.2, C700.2, C800.2, DEV0.1, DEV1.1, F300.GND@1, F300.GND@2, F300.GND@3, IC100.GND@1, IC100.GND@2, IC100.RGND, IC100.SA0, IC200.EN_N, IC200.NC, IC200.NC_2, IC200.PAD, IC200.VSS, IC200.VSS_2, IC300.EPAD, IC300.GND, IC300.GND_2, IC400.ADR0, IC400.ADR1, IC500.AVSS, IC500.AVSS_2, IC500.DVSS, IC500.EPAD, IC600.ADD0, IC600.GND, IC700.GND, IC800.CTG, IC800.GND, IC800.QSTRT, LINK.2, PROG.4, R211.1, R222.1, R231.1, R300.1, R700.2, R711.1, S1.SH, X320G$2.P$1; no longer !WP.1, C102.2, C110.2, C120.2, C121.2, C150.1, C152.2, C300.1, F100.GND@1, F100.GND@2, F100.GND@3, IC100.EPAD, IC100.GND, IC100.GND_2, IC200.ADR0, IC200.ADR1, IC200.GND, IC300.A0, IC300.A1, IC300.A2, IC300.VSS, IC400.ADD0, PCB1.GND@14, PCB1.GND@20, PCB1.GND@25, PCB1.GND@30, PCB1.GND@34, PCB1.GND@39, PCB1.GND@6, PCB1.GND@9, R100.1, X120G$2.P$1
- net N$1: now also C351.1, C352.1, U$1.P$1; no longer !WP.2, IC300.WP, R300.1
- net N$2: now also F300.UNBAL, L350.1; no longer C151.1, C152.1, U$1.P$1
- net N$29: now also C320.1, IC300.XOSC_Q1, X320G$1.2; no longer C120.1, IC100.XOSC_Q1, X120G$1.2
- net N$34: now also F300.BAL@1, IC300.RF_N; no longer F100.BAL@1, IC100.RF_N
- net N$35: now also F300.BAL@2, IC300.RF_P; no longer F100.BAL@2, IC100.RF_P
- net N$36: now also C350.2, C351.2, L350.2; no longer C150.2, C151.2, L150.2
- net N$40: now also C310.1, IC300.DCOUPL; no longer C110.1, IC100.DCOUPL
- net N$41: now also IC300.RBIAS, R300.2; no longer IC100.RBIAS, R100.2
- net N$49: now also C321.1, IC300.XOSC_Q2, X320G$1.1; no longer C121.1, IC100.XOSC_Q2, X120G$1.1
- net VCC: now also !PROG.1, C300.1, C301.1, C302.1, C500.1, C501.1, C600.1, IC100.CS, IC100.VDD, IC100.VDD_IO, IC300.AVDD, IC300.AVDD_2, IC300.AVDD_3, IC300.AVDD_4, IC300.DGUARD, IC300.DVDD, IC400.VDD, IC500.AVCC, IC500.DVCC, IC600.V+, LINK.3, PROG.1, R500.2; no longer C102.1, C200.1, C300.2, IC100.AVDD, IC100.AVDD_2, IC100.AVDD_3, IC100.AVDD_4, IC100.DGUARD, IC100.DVDD, IC200.VDD, IC300.VCC, IC400.V+, PCB1.3V3@1, PCB1.3V3@17, R300.2, R310.2, R311.2

Commit message: CHG: Updated schematics and layout
Parts:
- R210: value 13M -> 7M32
- R230: value 7M8 -> 8M3
- R231: value 5M2 -> 4M7
Changed lines of the file:
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@@
 <?xml version="1.0" encoding="utf-8"?>
 <!DOCTYPE eagle SYSTEM "eagle.dtd">
-<eagle version="6.5.0">
+<eagle version="7.4.0">
 <drawing>
 <settings>
@@
 <attribute name="OC_FARNELL" value="unknown"/>
 </part>
-<part name="R210" library="rcl" deviceset="R-EU_" device="R0603" value="13M">
+<part name="R210" library="rcl" deviceset="R-EU_" device="R0603" value="7M32">
 <attribute name="MF" value=""/>
 <attribute name="MPN" value=""/>
@@
 <attribute name="OC_FARNELL" value="unknown"/>
 </part>
-<part name="R230" library="rcl" deviceset="R-EU_" device="R0603" value="7M8">
+<part name="R230" library="rcl" deviceset="R-EU_" device="R0603" value="8M3">
 <attribute name="MF" value=""/>
 <attribute name="MPN" value=""/>
@@
 <attribute name="OC_FARNELL" value="unknown"/>
 </part>
-<part name="R231" library="rcl" deviceset="R-EU_" device="R0603" value="5M2">
-<attribute name="MF" value=""/>
-<attribute name="MPN" value=""/>
+<part name="R231" library="rcl" deviceset="R-EU_" device="R0603" value="4M7">
+<attribute name="MF" value=""/>
+<attribute name="MPN" value=""/>

Commit message: CHG: fixed some issuses on pcb
Parts:
- added R712: 100k, rcl:R-EU_R0603
Connections:
- net GND: now also R712.1
- net TPL5111_DONE: now also R712.2
- net TPL5111_DRV: no longer IC500.P3.6/TB2.1/TB1CLK
Changed lines of the file:
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@@
 <part name="GND30" library="supply1" deviceset="GND" device=""/>
 <part name="C800" library="rcl" deviceset="C-EU" device="C0603" value="100n"/>
+<part name="R712" library="rcl" deviceset="R-EU_" device="R0603" value="100k">
+<attribute name="MF" value=""/>
+<attribute name="MPN" value=""/>
+<attribute name="OC_FARNELL" value="unknown"/>
+</part>
+<part name="GND33" library="supply1" deviceset="GND" device=""/>
 </parts>
 <sheets>
@@
 </segment>
 </net>
-<net name="TPL5111_DRV" class="0">
-<segment>
-<pinref part="IC500" gate="A" pin="P3.6/TB2.1/TB1CLK"/>
-<wire x1="226.06" y1="63.5" x2="241.3" y2="63.5" width="0.1524" layer="91"/>
-<label x="241.3" y="63.5" size="1.27" layer="95" xref="yes"/>
-</segment>
-</net>
 <net name="CC110L_GDO0" class="0">
 <segment>
@@
 </instance>
 <instance part="GND25" gate="1" x="50.8" y="96.52"/>
+<instance part="R712" gate="G$1" x="154.94" y="96.52" rot="R90">
+<attribute name="OC_FARNELL" x="154.94" y="96.52" size="1.778" layer="96" display="off"/>
+<attribute name="MF" x="154.94" y="96.52" size="1.778" layer="96" display="off"/>
+<attribute name="MPN" x="154.94" y="96.52" size="1.778" layer="96" display="off"/>
+</instance>
+<instance part="GND33" gate="1" x="154.94" y="86.36"/>
 </instances>
 <busses>
@@
 <pinref part="GND8" gate="1" pin="GND"/>
 <wire x1="73.66" y1="106.68" x2="73.66" y2="104.14" width="0.1524" layer="91"/>
-<wire x1="73.66" y1="104.14" x2="76.2" y2="104.14" width="0.1524" layer="91"/>
 <pinref part="IC700" gate="A" pin="GND"/>
-<wire x1="76.2" y1="104.14" x2="81.28" y2="104.14" width="0.1524" layer="91"/>
+<wire x1="73.66" y1="104.14" x2="81.28" y2="104.14" width="0.1524" layer="91"/>
 <wire x1="81.28" y1="104.14" x2="81.28" y2="99.06" width="0.1524" layer="91"/>
-<wire x1="99.06" y1="104.14" x2="81.28" y2="104.14" width="0.1524" layer="91"/>
+<wire x1="99.06" y1="104.14" x2="83.82" y2="104.14" width="0.1524" layer="91"/>
 <junction x="81.28" y="104.14"/>
 <pinref part="S1" gate="G$1" pin="SH"/>
-<wire x1="76.2" y1="121.92" x2="76.2" y2="104.14" width="0.1524" layer="91"/>
-<junction x="76.2" y="104.14"/>
+<wire x1="83.82" y1="104.14" x2="81.28" y2="104.14" width="0.1524" layer="91"/>
+<wire x1="76.2" y1="121.92" x2="83.82" y2="121.92" width="0.1524" layer="91"/>
+<wire x1="83.82" y1="121.92" x2="83.82" y2="104.14" width="0.1524" layer="91"/>
+<junction x="83.82" y="104.14"/>
 </segment>
 <segment>
@@
 <pinref part="GND25" gate="1" pin="GND"/>
 <wire x1="50.8" y1="99.06" x2="50.8" y2="109.22" width="0.1524" layer="91"/>
+</segment>
+<segment>
+<pinref part="R712" gate="G$1" pin="1"/>
+<pinref part="GND33" gate="1" pin="GND"/>
+<wire x1="154.94" y1="88.9" x2="154.94" y2="91.44" width="0.1524" layer="91"/>
 </segment>
 </net>
@@
 <segment>
 <pinref part="IC700" gate="A" pin="DONE"/>
-<wire x1="149.86" y1="104.14" x2="172.72" y2="104.14" width="0.1524" layer="91"/>
+<wire x1="149.86" y1="104.14" x2="154.94" y2="104.14" width="0.1524" layer="91"/>
 <label x="172.72" y="104.14" size="1.27" layer="95" xref="yes"/>
-</segment>
-</net>
+<pinref part="R712" gate="G$1" pin="2"/>
+<wire x1="154.94" y1="104.14" x2="172.72" y2="104.14" width="0.1524" layer="91"/>
+<wire x1="154.94" y1="101.6" x2="154.94" y2="104.14" width="0.1524" layer="91"/>
+<junction x="154.94" y="104.14"/>
+</segment>
+</net>
